File: Receiver-Transceiver/toslink receiver kicad project/ToslinkCNC_OneAxis.kicad_pcb (KiCad board)
At the start: 2 copper layers, 50 x 52 mm, 39 parts, among them P3 LIMIT SWITCH 1, P4 PoStep25-32 connector, P5 JTAG, SW1 DIP3, U1 TLV1117, U2 CFPS-9-50M, U3 XC9572XL, U4 DLT1111, U5 DLR1111, U6 DLT1111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

Commit message: Update
Parts:
- removed D2, D3: LED Green, VQFP44:LED_0603_HandSoldering
- removed P5: JTAG, Socket_Strips:Socket_Strip_Straight_1x06
- added J2: solder_bridge, solder_bridge:solder_bridge, B.Cu at (50.2, 107.4)
- added J3: solder_bridge, solder_bridge:solder_bridge, B.Cu at (50.2, 110.1)
- added J4: solder_bridge, solder_bridge:solder_bridge, B.Cu at (58.6, 121.1)
- added J5: solder_bridge, solder_bridge:solder_bridge, B.Cu at (58.7, 118.4)
- added P1: CONN_01X04, terminal_block_2_5mm_4pole:terminal_block_2_5mm_4pole, F.Cu at (46.9, 98.0)
- added P2: term_block, terminal_block_2_5mm:terminal_block_2_5mm, F.Cu at (46.9, 89.7)
- added Q1: RSR010N10FHATL, sot_32_standard:SOT-23, B.Cu at (50.5, 98.0)
- C3, C7, C9, R1, R5: moved to B.Cu
- P3: value LIMIT SWITCH 1 -> RPI_header; footprint Socket_Strips:Socket_Strip_Straight_1x02 -> Pin_Headers:Pin_Header_Straight_2x13
- R3: value 1K -> 10K; moved to B.Cu
- R4: value 1K -> 10K
- U7: value H11L1S-M -> TLP2704; footprint VQFP44:H11L1S-M -> TLP2704:TLP2704
- moved P3 49.3 mm to (87.6, 82.8), turned to 0 degrees
- moved R4 41.9 mm to (53.7, 116.3), turned to 0 degrees
- moved R3 30.5 mm to (52.9, 94.9)
- moved U7 17.5 mm to (57.7, 86.6)
- moved C1 15.0 mm to (57.2, 101.5), turned to 0 degrees
- moved R5 13.4 mm to (57.8, 86.6), turned to 180 degrees
- moved D4 12.3 mm to (81.8, 110.9)
- moved R2 12.3 mm to (77.1, 105.3)
- moved R6 12.3 mm to (77.1, 110.9)
- moved D1 12.3 mm to (81.7, 105.2)
- moved C10 12.2 mm to (55.1, 87.5), turned to 270 degrees
- moved U1 10.8 mm to (56.3, 105.9), turned to 180 degrees
- moved C6 9.85 mm to (62.9, 89.2), turned to 270 degrees
- moved C9 8.92 mm to (79.6, 78.5), turned to 90 degrees
- moved U2 8.55 mm to (63.9, 96.1)
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Connections:
- C10 pad 1: GND -> +5V
- C10 pad 2: +3V3 -> GND
- P3 pad 1: Net-(P3-Pad1) -> (no net)
- P3 pad 2: Net-(P3-Pad2) -> +5V
- P4 pad 9: +5V -> Net-(J4-Pad2)
- R1 pad 1: +5V -> Net-(J2-Pad2)
- R1 pad 2: Net-(P3-Pad2) -> Net-(R1-Pad2)
- R2 pad 2: RX_LED -> EN_LED
- R3 pad 1: Net-(D2-Pad2) -> GND
- R3 pad 2: TX1_LED -> TRIGGER
- R4 pad 1: Net-(D3-Pad2) -> +3V3
- R4 pad 2: TX2_LED -> ERROR
- R5 pad 1: +3V3 -> LIMIT
- R5 pad 2: LIMIT -> +5V
- R7 pad 2: AXIS_X -> AXIS_1
- R8 pad 2: AXIS_Y -> AXIS_2
- R9 pad 2: AXIS_Z -> AXIS_3
- SW1 pad 1: AXIS_X -> AXIS_1
- SW1 pad 2: AXIS_Y -> AXIS_2
- SW1 pad 3: AXIS_Z -> AXIS_3
- U3 pad 1: CLK -> ERROR
- U3 pad 12: CRC_ERROR -> GENERAL3
- U3 pad 13: AXIS_Y -> GENERAL6
- U3 pad 14: AXIS_X -> GENERAL5
- U3 pad 16: AXIS_Z -> (no net)
- U3 pad 18: (no net) -> GENERAL2
- U3 pad 19: LIMIT -> GENERAL1
- U3 pad 2: ENABLE -> STEP
- U3 pad 20: RX_LED -> UART_TX
- U3 pad 21: TX1_LED -> UART_RX
- U3 pad 22: TX2_LED -> I2C_SCL
- U3 pad 23: TOSLINK_TX1 -> I2C_SDA
- U3 pad 3: ERROR -> DIR
- U3 pad 32: (no net) -> TOSLINK_TX1
- U3 pad 37: (no net) -> TRIGGER
- U3 pad 38: (no net) -> LIMIT
- U3 pad 41: (no net) -> GENERAL4
- U3 pad 42: (no net) -> CRC_ERROR
- U3 pad 43: (no net) -> EN_LED
- U3 pad 44: (no net) -> CLK
- U3 pad 5: (no net) -> ENABLE
- U3 pad 6: (no net) -> AXIS_1
- U3 pad 7: STEP -> AXIS_2
- U3 pad 8: DIR -> AXIS_3
- U7 pad 1: Net-(P3-Pad1) -> Net-(R1-Pad2)
- U7 pad 2: GND -> (no net)
- U7 pad 3: (no net) -> Net-(P1-Pad3)
- U7 pad 4: LIMIT -> GND
- U7 pad 5: GND -> LIMIT
- U7 pad 6: +3V3 -> +5V
Routing:
- net TRIGGER: track 0.00 -> 54.4 mm, vias 0 -> 4
- net AXIS_X: track 53.4 -> 0.00 mm, vias 2 -> 0
- net +5V: track 74.0 -> 122.4 mm
- net +3V3: track 185.3 -> 142.2 mm, vias 4 -> 6
- net AXIS_1: track 0.00 -> 42.6 mm, vias 0 -> 2
- net GND: track 300.2 -> 342.4 mm, vias 4 -> 17
- net AXIS_Z: track 40.6 -> 0.00 mm, vias 2 -> 0
- net AXIS_2: track 0.00 -> 38.4 mm, vias 0 -> 2
- net ENABLE: track 24.7 -> 62.2 mm, vias 1 -> 3
- net GENERAL4: track 0.00 -> 37.1 mm, vias 0 -> 1
- net AXIS_Y: track 36.9 -> 0.00 mm, vias 2 -> 0
- net Net-(P1-Pad3): track 0.00 -> 27.9 mm, vias 0 -> 1
- net AXIS_3: track 0.00 -> 26.5 mm, vias 0 -> 2
- net GENERAL2: track 0.00 -> 20.1 mm, vias 0 -> 1
- net STEP: track 34.8 -> 54.5 mm, vias 1 -> 2
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Other:
- net class Default: clearance 0.254 -> 0.3; trace_width 0.381 -> 0.3
- rule trace_clearance: 0.254 -> 0.3
- rule trace_min: 0.2032 -> 0.3
- board text added: "1"
- board text added: "2"
- board text added: "3"
- board text added: "3V3"
- board text added: "5V"
- board text added: "AXIS SEL"
- board text added: "ENABLED"
- board text added: "L"
- board text added: "PWR"
- board text added: "T"
- board text added: "TRIGG/LIMIT"
- board text added: "Toslink CNC Transciever"
- board text added: "VCC"
- board text removed: "AXIS SEL 123"
- board text removed: "LIMIT SW"
- board text removed: "Toslink CNC Receiver"
