File: Receiver-Transceiver/toslink receiver kicad project/ToslinkCNC_OneAxis.sch (KiCad schematic (older format))
At the start: 34 parts, among them P3 LIMIT SWITCH 1, P4 PoStep25-32 connector, P5 JTAG, SW1 DIP3, U1 TLV1117, U2 CFPS-9-50M, U3 XC9572XL, U4 DLT1111, U5 DLR1111, U6 DLT1111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

Commit message: Update
Parts:
- removed D2, D3: LED Green, VQFP44:LED_0603_HandSoldering, symbol Led_Small
- removed P3: LIMIT SWITCH 1, Socket_Strips:Socket_Strip_Straight_1x02, symbol CONN_01X02
- removed P5: JTAG, Socket_Strips:Socket_Strip_Straight_1x06, symbol CONN_01X06
- removed U7: H11L1S-M, VQFP44:H11L1S-M, symbol H11L1S-M
- added J2, J3, J4, J5: solder_bridge, solder_bridge:solder_bridge, symbol solder_bridge
- added P1: CONN_01X04, terminal_block_2_5mm_4pole:terminal_block_2_5mm_4pole, symbol CONN_01X04
- added P2: term_block, terminal_block_2_5mm:terminal_block_2_5mm, symbol term_block
- added P3: RPI_header, Pin_Headers:Pin_Header_Straight_2x13, symbol RPI_header
- added Q1: RSR010N10FHATL, sot_32_standard:SOT-23, symbol RSR010N10FHATL
- added U7: TLP2704, TLP2704:TLP2704, symbol TLP2704
- R3, R4: value 1K -> 10K
Connections:
- net +3V3: now also R4.1, J3.1, J4.1; no longer C10.2, R5.1
- net +5V: now also C10.1, R5.2, J2.1, J5.1, P2.1 (VCC), P3.2 (5V), P3.4 (5V), U7.6 (VCC); no longer P4.9, R1.1
- net AXIS_1: now also U3.6 (PIN6); no longer U3.14 (PIN14)
- net AXIS_2: now also U3.7 (PIN7); no longer U3.13 (PIN13)
- net AXIS_3: now also U3.8 (PIN8); no longer U3.16 (PIN16)
- net CLK: now also U3.44 (I/O/GCK2); no longer U3.1 (I/O/GCK3)
- net CRC_ERROR: now also U3.42 (PIN42); no longer U3.12 (PIN12)
- net DIR: now also U3.3 (PIN3); no longer U3.8 (PIN8)
- net ENABLE: now also U3.5 (PIN5), P3.7 (GPIO4); no longer U3.2 (PIN2)
- net ERROR: now also R4.2, U3.1 (I/O/GCK3); no longer U3.3 (PIN3)
- net GND: now also C10.2, R3.1, P1.1 (P1), P2.2 (GND), P3.14 (GND), P3.20 (GND), P3.25 (GND), P3.6 (GND), P3.9 (GND), Q1.2 (S), U7.4 (GND); no longer C10.1
- net LIMIT: now also R5.1, U3.38 (PIN38), U7.5 (OUT); no longer R5.2, U3.19 (PIN19)
- net STEP: now also U3.2 (PIN2), P3.11 (GPIO17); no longer U3.7 (PIN7)
- net TCK: now also P3.23 (SPI_SCK)
- net TDI: now also P3.19 (SPI_MOSI)
- net TDO: now also P3.21 (SPI_MISO)
- net TMS: now also P3.24 (SPI_CE0_N)
- net TOSLINK_TX1: now also U3.32 (PIN32); no longer U3.23 (PIN23)
- net GENERAL2: now reaches U3.18 (PIN18)
- net GENERAL2: now also P3.18 (GPIO24)
- net TRIGGER: now reaches U3.37 (PIN37)
- net TRIGGER: now also R3.2, P3.12 (GPIO_18), Q1.1 (G)
- net GENERAL4: now reaches U3.41 (PIN41)
- net GENERAL4: now also P3.26 (SPI_CE1_N)
- net EN_LED: now reaches U3.43 (I/O/GCK1)
- net EN_LED: now also R2.2
- net at R1.2: now also U7.1 (A)
- net RX_LED renamed UART_TX
- net UART_TX: now also P3.10 (UART_RX); no longer R2.2
- net TX1_LED renamed UART_RX
- net UART_RX: now also P3.8 (UART_TX); no longer R3.2
- net TX2_LED renamed I2C_SCL
- net I2C_SCL: now also P3.5 (I2C_SCL); no longer R4.2
- new net: J4.2, J5.2, P4.9
- new net: J2.2, J3.2, P1.4 (P4), R1.1
- new net: P1.2 (P2), Q1.3 (D)
- new net: P1.3 (P3), U7.3 (K)
- new net GENERAL1: P3.16 (GPIO23), U3.19 (PIN19)
- new net GENERAL3: P3.22 (GPIO25), U3.12 (PIN12)
- new net GENERAL5: P3.13 (GPIO27), U3.14 (PIN14)
- new net GENERAL6: P3.15 (GPIO22), U3.13 (PIN13)
- new net I2C_SDA: P3.3 (I2C_SDA), U3.23 (PIN23)
- no-connect marks 19 -> 12
Other:
- note added: "Motor Enabled Indication"
- note added: "Trigger Signal Output"
- note removed: "Programming Interface"
- note removed: "Tsolink Transmission Indication"
- moved on the sheet: C1, C5, C6, P4, R1, R7, R8, R9, SW1, U1, U2, U3
