File: Transmitter/shield KiCAD project/toslink_arduino_shield.kicad_pcb (KiCad board)
At the start: 2 copper layers, 82.1 x 53.7 mm, 22 parts, among them J1 solder_bridge, J2 solder_bridge, J3 solder_bridge, J4 solder_bridge, J5 solder_bridge, J6 solder_bridge, J7 solder_bridge, J8 solder_bridge, J9 solder_bridge, P1 Arduino UNO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

Commit message: Update
Parts:
- removed G***: LOGO, opensource_hardware:OSHWLOGO0.75IN
- removed U1: SN74LV21APWR, SN74LV21APWR_ANDGate:SN74LV21APWR_ANDGate_tssop14
- P2: footprint toslink_pcb -> toslink_pcb:toslink_pcb
- R1, R2, R3, R4: value R -> 10K
Connections:
- P1 pad 8: ENABLE_ARDUINO -> ENABLE
- P3 pad 1: ENABLE_X -> ENABLE
- P4 pad 1: ENABLE_Y -> ENABLE
- P5 pad 1: ENABLE_Z -> ENABLE
- R1 pad 1: ENABLE_ARDUINO -> +5V
- R1 pad 2: +5V -> ENABLE
- R2 pad 1: ENABLE_X -> GND
- R2 pad 2: +5V -> TRIGGER3
- R3 pad 1: ENABLE_Y -> GND
- R3 pad 2: +5V -> TRIGGER2
- R4 pad 1: ENABLE_Z -> GND
- R4 pad 2: +5V -> TRIGGER1
Routing:
- net ENABLE: track 63.8 -> 158.3 mm, vias 4 -> 8
- net ENABLE_Z: track 54.5 -> 0.00 mm, vias 3 -> 0
- net ENABLE_ARDUINO: track 51.9 -> 0.00 mm, vias 2 -> 0
- net ENABLE_Y: track 43.3 -> 0.00 mm, vias 2 -> 0
- net ENABLE_X: track 32.9 -> 0.00 mm, vias 1 -> 0
- net GND: track 326.7 -> 359.1 mm, vias 5 -> 9
- net TRIGGER2: track 162.2 -> 169.6 mm
- net +5V: track 174.2 -> 166.8 mm, vias 8 -> 7
- net TRIGGER3: track 100.6 -> 104.9 mm
- net LIMIT_X: track 131.3 -> 134.4 mm
- net TRIGGER1: track 77.3 -> 79.9 mm, vias 6 -> 7
- net DIR_Z: track 99.7 -> 97.8 mm
